File: hardware/StarvedLogger_PCB/StarvedLogger_PCB.kicad_pcb (KiCad board)
At the start: 4 copper layers, 52 x 64.5 mm, 33 parts, among them J1 UART_DEBUG, J2 BAT_IN, J3 Conn_01x08, J4 Conn_01x04_Pin, J5 Conn_01x03_Pin, J6 Conn_01x04_Pin, J7 Conn_01x03_Pin, SW1 SW_Push, U1 ESP32-S3-MINI-1, U4 ASSR-1218, U5 ASSR-1218, U6 ASSR-1218, U7 ASSR-1218, U8 AP2112K-3.3

Commit message: Update StarvedLogger PCB design
Parts:
- added C5: 0.1µF, Capacitor_SMD:C_0603_1608Metric, F.Cu at (105.5, 42.0)
- added C6: 10pF, Capacitor_SMD:C_0603_1608Metric, F.Cu at (145.5, 61.0)
- added C7: 10pF, Capacitor_SMD:C_0603_1608Metric, F.Cu at (152.7, 63.5)
- added D2: LED, LED_SMD:LED_0603_1608Metric, F.Cu at (115.5, 55.0)
- added D3: LED, LED_SMD:LED_0603_1608Metric, F.Cu at (115.5, 51.5)
- added D4: LED, LED_SMD:LED_0603_1608Metric, F.Cu at (120.0, 55.0)
- added D5: LED, LED_SMD:LED_0603_1608Metric, F.Cu at (120.0, 51.5)
- added J10: Conn_01x05_Pin, Connector_PinHeader_2.54mm:PinHeader_1x05_P2.54mm_Vertical, F.Cu at (145.5, 65.5)
- added J8: Conn_01x06_Pin, Connector_PinHeader_2.54mm:PinHeader_1x06_P2.54mm_Vertical, F.Cu at (136.5, 71.2)
- added J9: USB_C_Receptacle_USB2.0_16P, Connector_USB:USB_C_Receptacle_Amphenol_12401610E4-2A_CircularHoles, F.Cu at (154.0, 55.5)
- added R16: 0.33k, Resistor_SMD:R_0603_1608Metric, F.Cu at (115.5, 58.0)
- added R17: 0.33k, Resistor_SMD:R_0603_1608Metric, F.Cu at (115.5, 48.5)
- added R18: 0.33k, Resistor_SMD:R_0603_1608Metric, F.Cu at (120.0, 58.0)
- added R19: 0.33k, Resistor_SMD:R_0603_1608Metric, F.Cu at (120.0, 48.5)
- added R2: 10k, Resistor_SMD:R_0603_1608Metric, F.Cu at (107.3, 49.0)
- added R20: 5.1k, Resistor_SMD:R_0603_1608Metric, F.Cu at (145.5, 58.0)
- added R21: 5.1k, Resistor_SMD:R_0603_1608Metric, F.Cu at (147.0, 48.0)
- added R22: 22R, Resistor_SMD:R_0603_1608Metric, F.Cu at (144.0, 55.0)
- added R23: 22R, Resistor_SMD:R_0603_1608Metric, F.Cu at (144.0, 52.0)
- added R24: 4.7k, Resistor_SMD:R_0603_1608Metric, F.Cu at (110.5, 39.5)
- added REF**: MountingHole_3.2mm_M3_Pad, MountingHole:MountingHole_3.2mm_M3_Pad, F.Cu at (91.0, 32.0)
- added REF**: MountingHole_3.2mm_M3_Pad, MountingHole:MountingHole_3.2mm_M3_Pad, F.Cu at (90.5, 83.5)
- added REF**: MountingHole_3.2mm_M3_Pad, MountingHole:MountingHole_3.2mm_M3_Pad, F.Cu at (154.5, 84.0)
- added SW2: SW_Push, Button_Switch_SMD:SW_SPST_TL3342, F.Cu at (137.0, 31.0)
- added U2: TMP117xxDRV, Package_SON:WSON-6-1EP_2x2mm_P0.65mm_EP1x1.6mm, F.Cu at (110.4, 42.5)
- moved J3 50.7 mm to (153.5, 28.0), turned to 0 degrees
- moved R1 17.3 mm to (144.5, 29.5), turned to 0 degrees
- moved C4 14.2 mm to (144.5, 32.0)
- moved C3 13.0 mm to (111.0, 29.0), turned to 180 degrees
- moved U1 11.7 mm to (122.5, 34.5)
- moved J1 6.07 mm to (142.1, 37.5), turned to -90 degrees
- moved R10 5.52 mm to (105.5, 39.0), turned to 0 degrees
- moved C1 5.01 mm to (100.5, 32.5)
- moved C2 5.01 mm to (109.8, 32.5)
- moved J2 5.01 mm to (99.8, 39.7)
- moved R11 5.01 mm to (105.5, 36.0)
- moved U8 5.01 mm to (105.3, 32.0)
- moved R12 3.81 mm to (106.2, 46.5)
- moved D1 2.74 mm to (102.5, 46.5)
Connections:
- R1 pad 1: +3.3V -> Net-(U1-EN)
- R1 pad 2: Net-(U1-EN) -> +3.3V
- U1 pad 16: unconnected-(U1-IO12-Pad16) -> Net-(J8-Pin_1)
- U1 pad 17: unconnected-(U1-IO13-Pad17) -> Net-(J8-Pin_2)
- U1 pad 18: unconnected-(U1-IO14-Pad18) -> Net-(J8-Pin_3)
- U1 pad 19: unconnected-(U1-IO15-Pad19) -> Net-(J8-Pin_4)
- U1 pad 20: unconnected-(U1-IO16-Pad20) -> Net-(J8-Pin_5)
- U1 pad 21: unconnected-(U1-IO17-Pad21) -> Net-(J8-Pin_6)
- U1 pad 23: unconnected-(U1-USB_D--Pad23) -> /USB-
- U1 pad 24: unconnected-(U1-USB_D+-Pad24) -> /USB+
- U1 pad 29: unconnected-(U1-IO34-Pad29) -> Net-(J10-Pin_5)
- U1 pad 30: unconnected-(U1-IO48-Pad30) -> Net-(J10-Pin_1)
- U1 pad 35: unconnected-(U1-IO39-Pad35) -> Net-(J10-Pin_4)
- U1 pad 36: unconnected-(U1-IO40-Pad36) -> Net-(J10-Pin_3)
- U1 pad 37: unconnected-(U1-IO41-Pad37) -> Net-(J10-Pin_2)
- U1 pad 5: unconnected-(U1-IO1-Pad5) -> /ALERT
Routing:
- net GND: track 231.3 -> 388.4 mm, vias 13 -> 16
- net +3.3V: track 214.1 -> 286.2 mm, vias 6 -> 5
- net Net-(J10-Pin_2): track 0.00 -> 44.1 mm, vias 0 -> 1
- net Net-(J10-Pin_4): track 0.00 -> 43.8 mm, vias 0 -> 2
- net Net-(J10-Pin_5): track 0.00 -> 43.5 mm, vias 0 -> 1
- net Net-(J10-Pin_3): track 0.00 -> 41.9 mm, vias 0 -> 2
- net Net-(J8-Pin_1): track 0.00 -> 38.5 mm
- net /6v Sensor: track 4.34 -> 40.5 mm, vias 0 -> 1
- net Net-(J8-Pin_2): track 0.00 -> 35.4 mm
- net Net-(J10-Pin_1): track 0.00 -> 32.9 mm, vias 0 -> 1
- net Net-(J8-Pin_3): track 0.00 -> 32.3 mm
- net /6v Sensor_1: track 6.72 -> 37.8 mm, vias 0 -> 2
- net /3.3v Sensor: track 6.50 -> 37.4 mm
- net Net-(J8-Pin_4): track 0.00 -> 29.3 mm
- net /USB-: track 0.00 -> 27.5 mm
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Other:
- board size 52 x 64.5 mm -> 72.2 x 61.8 mm
