File: hardware/StarvedLogger_PCB/StarvedLogger_PCB.kicad_sch (KiCad schematic)
At the start: 55 parts, among them J1 UART_DEBUG, J11 Conn_01x08_Pin, J2 BAT_IN, J3 Conn_01x08, J4 Conn_01x04_Pin, J5 Conn_01x03_Pin, J6 Conn_01x04_Pin, J7 Conn_01x03_Pin, J8 Conn_01x08_Pin, J9 USB_C_Receptacle_USB2.0_16P, SW1 SW_Push, SW2 SW_Push, U1 ESP32-S3-MINI-1, U2 TMP117xxDRV, U4 ASSR-1218, U5 ASSR-1218, U6 ASSR-1218, U7 ASSR-1218, U8 AP2112K-3.3

Commit message: Update StarvedLogger PCB design
Parts:
- removed J11, J8: Conn_01x08_Pin, Connector_PinHeader_2.54mm:PinHeader_1x08_P2.54mm_Vertical, symbol Connector:Conn_01x08_Pin
- added J10: Conn_01x05_Pin, Connector_PinHeader_2.54mm:PinHeader_1x05_P2.54mm_Vertical, symbol Connector:Conn_01x05_Pin
- added J8: Conn_01x06_Pin, Connector_PinHeader_2.54mm:PinHeader_1x06_P2.54mm_Vertical, symbol Connector:Conn_01x06_Pin
- D2, D3, D4, D5: footprint (none) -> LED_SMD:LED_0603_1608Metric
- J9: footprint (none) -> Connector_USB:USB_C_Receptacle_Amphenol_12401610E4-2A_CircularHoles
Connections:
- net GND: no longer U1.30 (IO48), U1.44 (IO46)
- net at U1.37 (IO41): now also J10.2 (Pin_2)
- net at U1.36 (IO40): now also J10.3 (Pin_3)
- net at U1.35 (IO39): now also J10.4 (Pin_4)
- net at U1.29 (IO34): now also J10.5 (Pin_5)
- net at U1.16 (IO12): now also J8.1 (Pin_1)
- net at U1.17 (IO13): now also J8.2 (Pin_2)
- net at U1.18 (IO14): now also J8.3 (Pin_3)
- net at U1.19 (IO15): now also J8.4 (Pin_4)
- net at U1.20 (IO16): now also J8.5 (Pin_5)
- net at U1.21 (IO17): now also J8.6 (Pin_6)
- new net: J10.1 (Pin_1), U1.30 (IO48)
- no-connect marks 3 -> 11
Other:
- moved on the sheet: J6, R17, U6
